File: power_board.brd (EAGLE design)
At the start: 160 x 100 mm, 18 parts, among them IC1 7805TV, IC2 7805TV, K1 G5LE, T1 2N3904, T2 2N3904, U1 ATTINY85V-10P

Commit message: PowerBoard PCB
Parts:
- moved T1 78.6 mm to (30.5, 6.35), turned to 90 degrees
- moved 5VCONSTANT 74.3 mm to (21.6, 52.1)
- moved T2 66.3 mm to (30.5, 14.0), turned to 91.2 degrees
- moved D1 61.3 mm to (29.2, 25.4), turned to 270 degrees
- moved C1 54.7 mm to (12.7, 43.2)
- moved IC1 53.6 mm to (16.5, 30.5), turned to 90 degrees
- moved C2 53.4 mm to (5.08, 43.2)
- moved C4 50.8 mm to (25.4, 36.8)
- moved FUSE2 49.6 mm to (8.89, 49.5), turned to 90 degrees
- moved IGN 48.6 mm to (10.2, 57.1)
- moved 5VDELAY 47.1 mm to (25.4, 52.1)
- moved C3 45.8 mm to (25.4, 33.0)
- moved GND 43.9 mm to (15.2, 57.1)
- moved IC2 40.8 mm to (21.6, 40.6), turned to 180 degrees
- moved K1 40.8 mm to (14.0, 12.7), turned to 180 degrees
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Routing:
- net GND: track 0.00 -> 121.3 mm
- net N$6: track 0.00 -> 73.0 mm
- net N$5: track 0.00 -> 67.2 mm
- net N$8: track 0.00 -> 40.1 mm
- net N$7: track 0.00 -> 35.0 mm
- net N$4: track 0.00 -> 34.5 mm
- net N$10: track 0.00 -> 30.6 mm
- net N$3: track 0.00 -> 19.9 mm
- net N$2: track 0.00 -> 7.25 mm
- net N$1: track 0.00 -> 6.81 mm
Other:
- board size 160 x 100 mm -> 36.8 x 64.4 mm
